File: eagle/ObstacleAvoidance/main.brd (EAGLE design)
At the start: 15 parts, among them IC1 L293D, X1 JST-XH-02-PIN-LONG-PAD, X2 JST-XH-02-PIN-LONG-PAD, X3 JST-XH-04-PIN-LONG-PAD

Commit message: Feat: Deleted buttons
Parts:
- removed IC1: L293D, st-microelectronics:DIL16
- removed J1, J2: (no value), jumper:05C
- added S1: TL46PO, switch:TL4XPO
- moved X3 3.81 mm to (81.3, 16.5)
Connections:
- removed net 12V-VCC2: IC1.8, J2.3
- removed net 8V: J1.3, X3.2
- new net N$11: S1.2
- new net N$5: S1.6
- new net N$6: S1.4
- new net N$8: S1.3
- new net N$9: S1.1
- net 12V: no longer J2.2
- net 5V: no longer IC1.16
- net 8V-1: now also S1.5; no longer J1.2, U$7.IN
- net GND: no longer IC1.12, IC1.13, IC1.4, IC1.5
- net IN1-A: no longer IC1.10
- net IN1-B: no longer IC1.7
- net IN2-A: no longer IC1.15
- net IN2-B: no longer IC1.2
- net N$1: no longer IC1.3
- net N$2: no longer IC1.6
- net N$3: no longer IC1.14
- net N$4: no longer IC1.11
- net PWM-A: no longer IC1.9
- net PWM-B: no longer IC1.1
Routing:
- net 8V: track 13.2 -> 0.00 mm
- net 8V-1: track 11.2 -> 0.00 mm
- net 12V-VCC2: track 51.1 -> 40.1 mm
- net 12V: track 25.7 -> 17.0 mm
Changed lines of the file:
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@@
 </groups>
 <elements>
-<element name="IC1" library="st-microelectronics" package="DIL16" value="L293D" x="125.73" y="48.26" smashed="yes">
-<attribute name="NAME" x="115.189" y="45.339" size="1.27" layer="25" ratio="10" rot="R90"/>
-<attribute name="VALUE" x="118.237" y="47.625" size="1.27" layer="27" ratio="10"/>
-</element>
 <element name="U$2" library="diy-modules" package="ULTRASONIC-HC-SR04#V" value="ULTRASONIC-HC-SR04#V" x="129.54" y="76.2" smashed="yes" rot="MR120">
 <attribute name="NAME" x="125.690515625" y="78.42249375" size="1.27" layer="26" rot="MR120" align="bottom-center"/>
@@
 <attribute name="VALUE" x="80.01" y="90.805" size="1.27" layer="28" rot="MR180" align="top-center"/>
 </element>
-<element name="J1" library="jumper" library_urn="urn:adsk.eagle:library:252" package="05C" package3d_urn="urn:adsk.eagle:package:15472/1" value="" x="64.77" y="16.51" smashed="yes" rot="MR180">
-<attribute name="NAME" x="64.77" y="15.367" size="1.27" layer="26" ratio="10" rot="MR180"/>
-<attribute name="POPULARITY" value="0" x="64.77" y="16.51" size="1.778" layer="28" rot="MR180" display="off"/>
-<attribute name="VALUE" x="67.2701" y="16.51" size="0.02" layer="28" rot="MR180"/>
-</element>
-<element name="J2" library="jumper" library_urn="urn:adsk.eagle:library:252" package="05C" package3d_urn="urn:adsk.eagle:package:15472/1" value="" x="92.71" y="16.51" smashed="yes" rot="MR180">
-<attribute name="NAME" x="90.17" y="12.827" size="1.27" layer="26" ratio="10" rot="MR180"/>
-<attribute name="POPULARITY" value="0" x="92.71" y="16.51" size="1.778" layer="28" rot="MR180" display="off"/>
-<attribute name="VALUE" x="95.2101" y="16.51" size="0.02" layer="28" rot="MR180"/>
-</element>
-<element name="X3" library="Rembrandt Electronics - JST XH Connectors v1-0" package="JST-XH-04-PACKAGE-LONG-PAD" value="JST-XH-04-PIN-LONG-PAD" x="81.28" y="20.32" smashed="yes" rot="R180">
-<attribute name="NAME" x="87.935" y="22.36" size="1.016" layer="25" ratio="10" rot="R270"/>
-<attribute name="VALUE" x="87.2825" y="16.4275" size="1.016" layer="27" ratio="10" rot="R180"/>
+<element name="X3" library="Rembrandt Electronics - JST XH Connectors v1-0" package="JST-XH-04-PACKAGE-LONG-PAD" value="JST-XH-04-PIN-LONG-PAD" x="81.28" y="16.51" smashed="yes" rot="R180">
+<attribute name="NAME" x="87.935" y="18.55" size="1.016" layer="25" ratio="10" rot="R270"/>
+<attribute name="VALUE" x="87.2825" y="12.6175" size="1.016" layer="27" ratio="10" rot="R180"/>
 </element>
 <element name="SV2" library="con-lstb" library_urn="urn:adsk.eagle:library:162" package="MA05-2" package3d_urn="urn:adsk.eagle:package:8329/1" value="" x="36.83" y="16.51" smashed="yes">
@@
 <attribute name="VALUE" x="36.83" y="12.319" size="1.27" layer="27" ratio="10"/>
 </element>
+<element name="S1" library="switch" library_urn="urn:adsk.eagle:library:380" package="TL4XPO" package3d_urn="urn:adsk.eagle:package:27746/1" value="TL46PO" x="81.28" y="25.4" smashed="yes" rot="R90">
+<attribute name="NAME" x="76.2" y="20.32" size="1.778" layer="25" rot="R90"/>
+<attribute name="POPULARITY" value="1" x="81.28" y="25.4" size="1.778" layer="27" rot="R90" display="off"/>
+<attribute name="VALUE" x="87.63" y="20.32" size="1.778" layer="27" rot="R90"/>
+</element>
 </elements>
 <signals>
-<signal name="8V">
-<contactref element="J1" pad="3"/>
-<contactref element="X3" pad="2"/>
-<wire x1="72.39" y1="16.51" x2="81.28" y2="16.51" width="1" layer="1"/>
-<wire x1="81.28" y1="16.51" x2="82.55" y2="17.78" width="1" layer="1"/>
-<wire x1="82.55" y1="17.78" x2="82.55" y2="20.32" width="1" layer="1"/>
-</signal>
 <signal name="12V">
 <contactref element="R2" pad="2"/>
-<contactref element="J2" pad="2"/>
 <contactref element="X3" pad="1"/>
-<wire x1="85.09" y1="20.32" x2="86.36" y2="21.59" width="1.5" layer="1"/>
-<wire x1="86.36" y1="21.59" x2="86.36" y2="33.02" width="1.5" layer="1"/>
-<wire x1="85.09" y1="20.32" x2="92.71" y2="20.32" width="1.5" layer="1"/>
-<wire x1="92.71" y1="20.32" x2="95.25" y2="17.78" width="1.5" layer="1"/>
-<wire x1="95.25" y1="17.78" x2="95.25" y2="16.51" width="1.5" layer="1"/>
+<wire x1="85.09" y1="16.51" x2="86.36" y2="17.78" width="1.5" layer="1"/>
+<wire x1="86.36" y1="17.78" x2="86.36" y2="33.02" width="1.5" layer="1"/>
 </signal>
 <signal name="GND">
 <contactref element="U$7" pad="GND"/>
-<contactref element="IC1" pad="5"/>
-<contactref element="IC1" pad="4"/>
-<contactref element="IC1" pad="12"/>
-<contactref element="IC1" pad="13"/>
 <contactref element="U$3" pad="4"/>
 <contactref element="U$2" pad="4"/>
@@
 <wire x1="102.87" y1="73.66" x2="102.87" y2="58.42" width="1" layer="1"/>
 <wire x1="97.79" y1="50.165" x2="97.79" y2="36.83" width="1" layer="1"/>
+<wire x1="102.87" y1="73.66" x2="131.445" y2="79.49955625" width="0" layer="19" extent="1-1"/>
+<wire x1="97.79" y1="50.165" x2="102.87" y2="58.42" width="0" layer="19" extent="1-1"/>
+<wire x1="86.36" y1="35.56" x2="97.79" y2="36.83" width="0" layer="19" extent="1-1"/>
+<wire x1="83.82" y1="72.39" x2="102.87" y2="73.66" width="0" layer="19" extent="1-1"/>
+<wire x1="77.47" y1="16.51" x2="86.36" y2="35.56" width="0" layer="19" extent="1-1"/>
+<wire x1="57.15" y1="20.32" x2="77.47" y2="16.51" width="0" layer="19" extent="1-1"/>
+<wire x1="49.53" y1="15.24" x2="55.753" y2="14.097" width="0" layer="19" extent="1-1"/>
+<wire x1="41.91" y1="15.24" x2="49.53" y2="15.24" width="0" layer="19" extent="1-1"/>
+<wire x1="24.33" y1="34.28" x2="41.91" y2="15.24" width="0" layer="19" extent="1-1"/>
+<wire x1="55.88" y1="71.12" x2="83.82" y2="72.39" width="0" layer="19" extent="1-1"/>
+<wire x1="33.655" y1="72.900440625" x2="44.45" y2="77.47" width="0" layer="19" extent="1-1"/>
 </signal>
 <signal name="5V">
-<contactref element="IC1" pad="16"/>
 <contactref element="U$1" pad="30"/>
 <via x="102.87" y="50.165" extent="1-16" drill="0.4" diameter="2"/>
@@
 </signal>
 <signal name="N$1">
-<contactref element="IC1" pad="3"/>
 <via x="121.92" y="39.259715625" extent="1-16" drill="0.35" diameter="2"/>
 <contactref element="X1" pad="2"/>
@@
 </signal>
 <signal name="N$2">
-<contactref element="IC1" pad="6"/>
 <wire x1="126.999996875" y1="39.369996875" x2="127" y2="39.259715625" width="1" layer="1"/>
 <via x="127" y="39.259715625" extent="1-16" drill="0.35" diameter="2"/>
@@
 </signal>
 <signal name="N$3">
-<contactref element="IC1" pad="14"/>
 <via x="121.92" y="57.15" extent="1-16" drill="0.35" diameter="2"/>
 <contactref element="X2" pad="1"/>
@@
 </signal>
 <signal name="N$4">
-<contactref element="IC1" pad="11"/>
 <via x="128.27" y="57.15" extent="1-16" drill="0.35" diameter="2"/>
 <contactref element="X2" pad="2"/>
@@
 </signal>
 <signal name="IN1-B">
-<contactref element="IC1" pad="7"/>
 <contactref element="U$1" pad="6"/>
 <wire x1="49.1" y1="44.44" x2="57.16" y2="44.44" width="1" layer="16"/>
@@
 </signal>
 <signal name="IN2-A">
-<contactref element="IC1" pad="15"/>
 <contactref element="U$1" pad="9"/>
 <wire x1="49.1" y1="52.06" x2="92.7" y2="52.06" width="1" layer="16"/>
@@
 </signal>
 <signal name="IN1-A">
-<contactref element="IC1" pad="10"/>
 <contactref element="U$1" pad="10"/>
 <wire x1="49.1" y1="54.6" x2="90.16" y2="54.6" width="1" layer="16"/>
@@
 </signal>
 <signal name="PWM-A">
-<contactref element="IC1" pad="9"/>
 <contactref element="U$1" pad="11"/>
 <wire x1="134.62" y1="58.42" x2="127" y2="66.04" width="1" layer="16"/>
@@
 </signal>
 <signal name="IN2-B">
-<contactref element="IC1" pad="2"/>
 <contactref element="U$1" pad="7"/>
 <wire x1="49.1" y1="46.98" x2="59.7" y2="46.98" width="1" layer="16"/>
@@
 </signal>
 <signal name="PWM-B">
-<contactref element="IC1" pad="1"/>
 <contactref element="U$1" pad="8"/>
 <wire x1="49.1" y1="49.52" x2="62.24" y2="49.52" width="1" layer="16"/>
@@
 </signal>
 <signal name="12V-VCC2">
-<contactref element="IC1" pad="8"/>
-<contactref element="J2" pad="3"/>
 <via x="109.22" y="21.59" extent="1-16" drill="0.35" diameter="2"/>
-<wire x1="100.33" y1="16.51" x2="104.14" y2="16.51" width="1.5" layer="1"/>
-<wire x1="104.14" y1="16.51" x2="109.22" y2="21.59" width="1.5" layer="1"/>
 <wire x1="109.22" y1="21.59" x2="120.65" y2="21.59" width="1.5" layer="16"/>
 <wire x1="120.65" y1="21.59" x2="134.62" y2="35.56" width="1.5" layer="16"/>
@@
 </signal>
 <signal name="8V-1">
-<contactref element="U$7" pad="IN"/>
-<contactref element="J1" pad="2"/>
-<wire x1="67.31" y1="16.51" x2="64.77" y2="19.05" width="1" layer="1"/>
-<wire x1="60.071" y1="19.05" x2="58.039" y2="17.018" width="1" layer="1"/>
-<wire x1="64.77" y1="19.05" x2="60.071" y2="19.05" width="1" layer="1"/>
+<contactref element="S1" pad="5"/>
 </signal>
 <signal name="OUT4">
@@
 </polygon>
 </signal>
+<signal name="N$5">
+<contactref element="S1" pad="6"/>
+</signal>
+<signal name="N$6">
+<contactref element="S1" pad="4"/>
+</signal>
+<signal name="N$8">
+<contactref element="S1" pad="3"/>
+</signal>
+<signal name="N$9">
+<contactref element="S1" pad="1"/>
+</signal>
+<signal name="N$11">
+<contactref element="S1" pad="2"/>
+</signal>
 </signals>

Commit message: Feat: PCB printing files
Parts:
- added IC1: L293D, st-microelectronics:DIL16
- moved U$2 2.54 mm to (129.5, 73.7)
- moved U$3 2.54 mm to (31.8, 73.7)
Connections:
- removed net N$11: S1.2
- removed net N$5: S1.6
- removed net N$6: S1.4
- removed net N$8: S1.3
- removed net N$9: S1.1
- new net 12V-VCC: IC1.8, S1.5
- new net 8V: S1.1, X3.2
- net 12V: now also S1.6
- net 5V: now also IC1.16
- net 8V-1: now also S1.2, U$7.IN; no longer S1.5
- net GND: now also IC1.12, IC1.13, IC1.4, IC1.5
- net IN1-A: now also IC1.10
- net IN1-B: now also IC1.7
- net IN2-A: now also IC1.15
- net IN2-B: now also IC1.2
- net N$1: now also IC1.3
- net N$2: now also IC1.6
- net N$3: now also IC1.14
- net N$4: now also IC1.11
- net PWM-A: now also IC1.9
- net PWM-B: now also IC1.1
Routing:
- net 12V-VCC: track 0.00 -> 67.1 mm, vias 0 -> 1
- net 12V-VCC2: track 40.1 -> 0.00 mm, vias 1 -> 0
- net 8V-1: track 0.00 -> 24.2 mm
- net 8V: track 0.00 -> 7.93 mm
- net 3.3V: track 190.8 -> 185.9 mm
- net 12V: track 17.0 -> 21.7 mm
- net ECHO-L: track 27.5 -> 25.7 mm
- net ECHO-R: track 86.0 -> 84.2 mm
- net TRIG-R: track 84.1 -> 83.0 mm
